File: rp2040-ISO-keyboard-pcb.kicad_pcb (KiCad board)
At the start: 2 copper layers, 3.6 x 3.3 mm, 399 parts, among them J1 USB_C_Receptacle_USB2.0, SW01 Boot, SW02 Boot, SW1 SW_HS, SW10 SW_HS, SW11 SW_HS, SW12 SW_HS, SW13 SW_HS, SW14 SW_HS, SW15 SW_HS, SW16 SW_HS, SW17 SW_HS, SW18 SW_HS, SW19 SW_HS, SW2 SW_HS, SW20 SW_HS, SW21 SW_HS, SW22 SW_HS, SW23 SW_HS, SW24 SW_HS, SW25 SW_HS, SW26 SW_HS, SW27 SW_HS, SW28 SW_HS, SW29 SW_HS, SW3 SW_HS, SW30 SW_HS, SW31 SW_HS, SW32 SW_HS, SW33 SW_HS, SW34 SW_HS, SW35 SW_HS, SW36 SW_HS, SW37 SW_HS, SW38 SW_HS, SW39 SW_HS, SW4 SW_HS, SW40 SW_HS, SW41 SW_HS, SW42 SW_HS, SW43 SW_HS, SW44 SW_HS, SW45 SW_HS, SW46 SW_HS, SW47 SW_HS, SW48 SW_HS, SW49 SW_HS, SW5 SW_HS, SW50 SW_HS, SW51 SW_HS, SW52 SW_HS, SW53 SW_HS, SW54 SW_HS, SW55 SW_HS, SW56 SW_HS, SW57 SW_HS, SW58 SW_HS, SW59 SW_HS, SW6 SW_HS, SW60 SW_HS, SW61 SW_HS, SW62 SW_HS, SW63 SW_HS, SW64 SW_HS, SW65 SW_HS, SW66 SW_HS, SW67 SW_HS, SW68 SW_HS, SW69 SW_HS, SW7 SW_HS, SW70 SW_HS, SW71 SW_HS, SW72 SW_HS, SW73 SW_HS, SW74 SW_HS, SW75 SW_HS, SW76 SW_HS, SW77 SW_HS, SW78 SW_HS, SW79 SW_HS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

Commit message: placed switches and LEDs
Parts:
- removed the C88 at (-38.8, -1.62)
- removed C89, C90: 0.1uf, Capacitor_SMD:C_0402_1005Metric
- removed the D64 at (-351.9, 188.7)
- removed the D78 at (-174.1, 26.0)
- removed the LED88 at (-344.6, 270.1)
- removed LED89, LED90: MX_SK6812MINI-E, marbastlib-mx:LED_MX_6028R
- removed the SW64 at (-243.8, 84.9)
- removed the SW78 at (-142.9, 84.2)
- moved LED15 719.2 mm to (-64.3, -313.1), turned to 0 degrees
- moved LED16 693.9 mm to (-45.2, -313.1), turned to 0 degrees
- moved LED49 690.0 mm to (-64.3, -270.2), turned to 0 degrees
- moved LED33 645.6 mm to (-45.2, -289.2), turned to 0 degrees
- moved LED8 644.6 mm to (-211.9, -313.1), turned to 0 degrees
- moved LED34 633.7 mm to (-369.1, -270.2), turned to 0 degrees
- moved LED24 632.3 mm to (-240.5, -289.2), turned to 0 degrees
- moved LED6 630.7 mm to (-250.0, -313.1), turned to 0 degrees
- moved LED48 627.4 mm to (-83.3, -270.2), turned to 0 degrees
- moved LED31 626.2 mm to (-83.3, -289.2), turned to 0 degrees
- moved LED4 624.5 mm to (-297.7, -313.1), turned to 0 degrees
- moved LED14 624.3 mm to (-83.3, -313.1), turned to 0 degrees
- moved LED28 622.8 mm to (-164.3, -289.2), turned to 0 degrees
- moved LED35 622.5 mm to (-345.3, -270.2), turned to 0 degrees
- moved LED12 611.5 mm to (-126.2, -313.1), turned to 0 degrees
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- renumbered C81 to C82, C82 to C83, C83 to C84, C84 to C85, C85 to C86, C86 to C87, C87 to C88, D65 to D64, D66 to D65, D67 to D66, D68 to D67, D69 to D68, D70 to D69, D71 to D70, D72 to D71, D73 to D72, D74 to D73, D75 to D74, D76 to D75, D77 to D76, D79 to D77, D80 to D78, D81 to D79, D82 to D80, D83 to D81, D84 to D82, D85 to D83, D86 to D84, D87 to D85, D88 to D86, D89 to D87, D90 to D88, LED81 to LED82, LED82 to LED83, LED83 to LED84, LED84 to LED85, LED85 to LED86, LED86 to LED87, LED87 to LED88, SW65 to SW64, SW66 to SW65, SW67 to SW66, SW68 to SW67, SW69 to SW68, SW70 to SW69, SW71 to SW70, SW72 to SW71, SW73 to SW72, SW74 to SW73, SW75 to SW74, SW76 to SW75, SW77 to SW76, SW79 to SW77, SW80 to SW78, SW81 to SW79, SW82 to SW80, SW83 to SW81, SW84 to SW82, SW85 to SW83, SW86 to SW84, SW87 to SW85, SW88 to SW86, SW89 to SW87, SW90 to SW88, SW01 to btn1, SW02 to btn2
Connections:
- LED88 pad 2: Net-(LED87-Pad2) (its old number) -> unconnected-(LED88-Pad2)

Commit message: some layouts done
Parts:
- removed the C10 at (-27.3, -3.59)
- removed the C11 at (-30.2, 4.29)
- removed the C12 at (-35.9, 4.29)
- removed the C13 at (-30.2, 2.32)
- removed the C14 at (-12.9, -1.62)
- removed the C15 at (-24.4, 8.23)
- removed the C20 at (-38.8, 2.32)
- removed the C21 at (-27.3, -5.56)
- removed the C22 at (-30.2, 10.2)
- removed the C23 at (-35.9, 8.23)
- removed the C24 at (-24.4, -3.59)
- removed C25, C26, C27, C28, C29, C30, C31, C32, C33, C34, C35, C36, C37, C38, C39, C40, C41, C42, C43, C44, C45, C46, C47, C48, C49, C50, C51, C52, C53, C54, C55, C56, C57, C58, C59, C60, C61, C62, C63, C64, C65, C66, C67, C68, C69, C70, C71, C72, C73, C74, C75, C76, C77, C78, C79, C80, C82, C83, C84, C85, C86, C87, C88: 0.1uf, Capacitor_SMD:C_0402_1005Metric
- removed the C4 at (-21.6, -3.59)
- removed the C5 at (-30.2, 0.35)
- removed the C6 at (-15.8, 4.29)
- removed the C7 at (-27.3, 0.35)
- removed the C8 at (-21.6, 4.29)
- removed the C9 at (-18.7, -5.56)
- removed LED1, LED10, LED11, LED12, LED13, LED14, LED15, LED16, LED17, LED18, LED19, LED2, LED20, LED21, LED22, LED23, LED24, LED25, LED26, LED27, LED28, LED29, LED3, LED30, LED31, LED32, LED33, LED34, LED35, LED36, LED37, LED38, LED39, LED4, LED40, LED41, LED42, LED43, LED44, LED45, LED46, LED47, LED48, LED49, LED5, LED50, LED51, LED52, LED53, LED54, LED55, LED56, LED57, LED58, LED59, LED6, LED60, LED61, LED62, LED63, LED64, LED65, LED66, LED67, LED68, LED69, LED7, LED70, LED71, LED72, LED73, LED74, LED75, LED76, LED77, LED78, LED79, LED8, LED80, LED82, LED83, LED84, LED85, LED86, LED87, LED88, LED9: MX_SK6812MINI-E, marbastlib-mx:LED_MX_6028R
- removed the U5 at (-392.9, 357.9)
- added J2: Conn_01x04, Connector_PinHeader_2.54mm:PinHeader_1x04_P2.54mm_Vertical, B.Cu at (-200.6, -187.0)
- added R10: 100k, Resistor_SMD:R_0603_1608Metric, B.Cu at (-208.3, -176.4)
- added R11: 20k, Resistor_SMD:R_0603_1608Metric, B.Cu at (-204.3, -175.9)
- added R13: 10k, Resistor_SMD:R_0603_1608Metric, B.Cu at (-230.2, -188.1)
- added R14: 51k, Resistor_SMD:R_0603_1608Metric, B.Cu at (-208.9, -178.9)
- added R16: 20k, Resistor_SMD:R_0603_1608Metric, B.Cu at (-222.2, -183.1)
- added R17: 20k, Resistor_SMD:R_0603_1608Metric, B.Cu at (-208.3, -173.8)
- added R18: 51k, Resistor_SMD:R_0603_1608Metric, B.Cu at (-226.2, -185.6)
- added R19: 20k, Resistor_SMD:R_0603_1608Metric, B.Cu at (-224.9, -180.6)
- added R2: 2k, Resistor_SMD:R_0603_1608Metric, B.Cu at (-218.2, -183.1)
- added R20: 20k, Resistor_SMD:R_0603_1608Metric, B.Cu at (-214.1, -188.1)
- added R21: 51k, Resistor_SMD:R_0603_1608Metric, B.Cu at (-214.1, -185.6)
- added R22: 20k, Resistor_SMD:R_0603_1608Metric, B.Cu at (-218.2, -185.6)
- added R23: 20k, Resistor_SMD:R_0603_1608Metric, B.Cu at (-222.2, -185.6)
- added R24: 51k, Resistor_SMD:R_0603_1608Metric, B.Cu at (-216.9, -180.6)
- added R25: 20k, Resistor_SMD:R_0603_1608Metric, B.Cu at (-214.1, -183.1)
- added R26: 20k, Resistor_SMD:R_0603_1608Metric, B.Cu at (-200.2, -175.9)
- added R27: 51k, Resistor_SMD:R_0603_1608Metric, B.Cu at (-216.3, -173.8)
- added R28: 20k, Resistor_SMD:R_0603_1608Metric, B.Cu at (-226.2, -183.1)
- added R29: 20k, Resistor_SMD:R_0603_1608Metric, B.Cu at (-212.9, -178.9)
- added R3: 2k, Resistor_SMD:R_0603_1608Metric, B.Cu at (-226.2, -188.1)
- added R30: 51k, Resistor_SMD:R_0603_1608Metric, B.Cu at (-216.3, -176.4)
- added R31: 20k, Resistor_SMD:R_0603_1608Metric, B.Cu at (-200.2, -170.8)
- added R32: 20k, Resistor_SMD:R_0603_1608Metric, B.Cu at (-204.9, -178.9)
- added R33: 51k, Resistor_SMD:R_0603_1608Metric, B.Cu at (-204.3, -170.8)
- added R34: 20k, Resistor_SMD:R_0603_1608Metric, B.Cu at (-200.2, -173.4)
- added R35: 20k, Resistor_SMD:R_0603_1608Metric, B.Cu at (-208.3, -171.3)
- added R36: 51k, Resistor_SMD:R_0603_1608Metric, B.Cu at (-222.2, -188.1)
- added R37: 20k, Resistor_SMD:R_0603_1608Metric, B.Cu at (-212.3, -173.8)
- added R38: 20k, Resistor_SMD:R_0603_1608Metric, B.Cu at (-220.3, -178.1)
- added R39: 51k, Resistor_SMD:R_0603_1608Metric, B.Cu at (-218.2, -188.1)
- added R6: 20k, Resistor_SMD:R_0603_1608Metric, B.Cu at (-212.3, -171.3)
- added R7: 20k, Resistor_SMD:R_0603_1608Metric, B.Cu at (-220.9, -180.6)
- added R9: 20k, Resistor_SMD:R_0603_1608Metric, B.Cu at (-204.3, -173.4)
- added RGB1: LED_ABGR, marbastlib-various:MHT151RGBCT-RGB-Reverse-Mount-1206, B.Cu at (-406.4, -317.8)
- added RGB10: LED_ABGR, marbastlib-various:MHT151RGBCT-RGB-Reverse-Mount-1206, B.Cu at (-206.4, -317.8)
- added RGB11: LED_ABGR, marbastlib-various:MHT151RGBCT-RGB-Reverse-Mount-1206, B.Cu at (-177.8, -317.8)
- added RGB12: LED_ABGR, marbastlib-various:MHT151RGBCT-RGB-Reverse-Mount-1206, B.Cu at (-158.7, -317.8)
- added RGB13: LED_ABGR, marbastlib-various:MHT151RGBCT-RGB-Reverse-Mount-1206, B.Cu at (-139.7, -317.8)
- added RGB14: LED_ABGR, marbastlib-various:MHT151RGBCT-RGB-Reverse-Mount-1206, B.Cu at (-115.9, -317.8)
- added RGB15: LED_ABGR, marbastlib-various:MHT151RGBCT-RGB-Reverse-Mount-1206, B.Cu at (-96.8, -317.8)
- added RGB16: LED_ABGR, marbastlib-various:MHT151RGBCT-RGB-Reverse-Mount-1206, B.Cu at (-77.8, -317.8)
- added RGB17: LED_ABGR, marbastlib-various:MHT151RGBCT-RGB-Reverse-Mount-1206, B.Cu at (-406.4, -294.0)
- added RGB18: LED_ABGR, marbastlib-various:MHT151RGBCT-RGB-Reverse-Mount-1206, B.Cu at (-387.3, -294.0)
- added RGB19: LED_ABGR, marbastlib-various:MHT151RGBCT-RGB-Reverse-Mount-1206, B.Cu at (-368.3, -294.0)
- added RGB2: LED_ABGR, marbastlib-various:MHT151RGBCT-RGB-Reverse-Mount-1206, B.Cu at (-377.8, -317.8)
- added RGB20: LED_ABGR, marbastlib-various:MHT151RGBCT-RGB-Reverse-Mount-1206, B.Cu at (-349.2, -294.0)
- added RGB21: LED_ABGR, marbastlib-various:MHT151RGBCT-RGB-Reverse-Mount-1206, B.Cu at (-330.2, -294.0)
- added RGB22: LED_ABGR, marbastlib-various:MHT151RGBCT-RGB-Reverse-Mount-1206, B.Cu at (-311.1, -294.0)
- added RGB23: LED_ABGR, marbastlib-various:MHT151RGBCT-RGB-Reverse-Mount-1206, B.Cu at (-292.1, -294.0)
- added RGB24: LED_ABGR, marbastlib-various:MHT151RGBCT-RGB-Reverse-Mount-1206, B.Cu at (-273.0, -294.0)
- added RGB25: LED_ABGR, marbastlib-various:MHT151RGBCT-RGB-Reverse-Mount-1206, B.Cu at (-254.0, -294.0)
- added RGB26: LED_ABGR, marbastlib-various:MHT151RGBCT-RGB-Reverse-Mount-1206, B.Cu at (-234.9, -294.0)
- added RGB27: LED_ABGR, marbastlib-various:MHT151RGBCT-RGB-Reverse-Mount-1206, B.Cu at (-215.9, -294.0)
- added RGB28: LED_ABGR, marbastlib-various:MHT151RGBCT-RGB-Reverse-Mount-1206, B.Cu at (-196.8, -294.0)
- added RGB29: LED_ABGR, marbastlib-various:MHT151RGBCT-RGB-Reverse-Mount-1206, B.Cu at (-177.8, -294.0)
- added RGB3: LED_ABGR, marbastlib-various:MHT151RGBCT-RGB-Reverse-Mount-1206, B.Cu at (-358.8, -317.8)
- added RGB30: LED_ABGR, marbastlib-various:MHT151RGBCT-RGB-Reverse-Mount-1206, B.Cu at (-149.2, -294.0)
- added RGB31: LED_ABGR, marbastlib-various:MHT151RGBCT-RGB-Reverse-Mount-1206, B.Cu at (-115.9, -294.0)
- added RGB32: LED_ABGR, marbastlib-various:MHT151RGBCT-RGB-Reverse-Mount-1206, B.Cu at (-96.8, -294.0)
- added RGB33: LED_ABGR, marbastlib-various:MHT151RGBCT-RGB-Reverse-Mount-1206, B.Cu at (-77.8, -294.0)
- added RGB34: LED_ABGR, marbastlib-various:MHT151RGBCT-RGB-Reverse-Mount-1206, B.Cu at (-401.6, -275.0)
- added RGB35: LED_ABGR, marbastlib-various:MHT151RGBCT-RGB-Reverse-Mount-1206, B.Cu at (-377.8, -275.0)
- added RGB36: LED_ABGR, marbastlib-various:MHT151RGBCT-RGB-Reverse-Mount-1206, B.Cu at (-358.8, -275.0)
- added RGB37: LED_ABGR, marbastlib-various:MHT151RGBCT-RGB-Reverse-Mount-1206, B.Cu at (-339.7, -275.0)
- added RGB38: LED_ABGR, marbastlib-various:MHT151RGBCT-RGB-Reverse-Mount-1206, B.Cu at (-320.7, -275.0)
- added RGB39: LED_ABGR, marbastlib-various:MHT151RGBCT-RGB-Reverse-Mount-1206, B.Cu at (-301.6, -275.0)
- added RGB4: LED_ABGR, marbastlib-various:MHT151RGBCT-RGB-Reverse-Mount-1206, B.Cu at (-339.7, -317.8)
- added RGB40: LED_ABGR, marbastlib-various:MHT151RGBCT-RGB-Reverse-Mount-1206, B.Cu at (-282.6, -275.0)
- added RGB41: LED_ABGR, marbastlib-various:MHT151RGBCT-RGB-Reverse-Mount-1206, B.Cu at (-263.5, -275.0)
- added RGB42: LED_ABGR, marbastlib-various:MHT151RGBCT-RGB-Reverse-Mount-1206, B.Cu at (-244.5, -275.0)
- added RGB43: LED_ABGR, marbastlib-various:MHT151RGBCT-RGB-Reverse-Mount-1206, B.Cu at (-225.4, -275.0)
- added RGB44: LED_ABGR, marbastlib-various:MHT151RGBCT-RGB-Reverse-Mount-1206, B.Cu at (-206.4, -275.0)
- added RGB45: LED_ABGR, marbastlib-various:MHT151RGBCT-RGB-Reverse-Mount-1206, B.Cu at (-187.3, -275.0)
- added RGB46: LED_ABGR, marbastlib-various:MHT151RGBCT-RGB-Reverse-Mount-1206, B.Cu at (-168.3, -275.0)
- added RGB47: LED_ABGR, marbastlib-various:MHT151RGBCT-RGB-Reverse-Mount-1206, B.Cu at (-142.1, -265.4)
- added RGB48: LED_ABGR, marbastlib-various:MHT151RGBCT-RGB-Reverse-Mount-1206, B.Cu at (-115.9, -275.0)
- added RGB49: LED_ABGR, marbastlib-various:MHT151RGBCT-RGB-Reverse-Mount-1206, B.Cu at (-96.8, -275.0)
- added RGB5: LED_ABGR, marbastlib-various:MHT151RGBCT-RGB-Reverse-Mount-1206, B.Cu at (-311.1, -317.8)
- added RGB50: LED_ABGR, marbastlib-various:MHT151RGBCT-RGB-Reverse-Mount-1206, B.Cu at (-77.8, -275.0)
- added RGB51: LED_ABGR, marbastlib-various:MHT151RGBCT-RGB-Reverse-Mount-1206, B.Cu at (-399.2, -255.9)
- added RGB52: LED_ABGR, marbastlib-various:MHT151RGBCT-RGB-Reverse-Mount-1206, B.Cu at (-373.1, -255.9)
- added RGB53: LED_ABGR, marbastlib-various:MHT151RGBCT-RGB-Reverse-Mount-1206, B.Cu at (-354.0, -255.9)
- added RGB54: LED_ABGR, marbastlib-various:MHT151RGBCT-RGB-Reverse-Mount-1206, B.Cu at (-335.0, -255.9)
- added RGB55: LED_ABGR, marbastlib-various:MHT151RGBCT-RGB-Reverse-Mount-1206, B.Cu at (-315.9, -255.9)
- added RGB56: LED_ABGR, marbastlib-various:MHT151RGBCT-RGB-Reverse-Mount-1206, B.Cu at (-296.9, -255.9)
- added RGB57: LED_ABGR, marbastlib-various:MHT151RGBCT-RGB-Reverse-Mount-1206, B.Cu at (-277.8, -255.9)
- added RGB58: LED_ABGR, marbastlib-various:MHT151RGBCT-RGB-Reverse-Mount-1206, B.Cu at (-258.8, -255.9)
- added RGB59: LED_ABGR, marbastlib-various:MHT151RGBCT-RGB-Reverse-Mount-1206, B.Cu at (-239.7, -255.9)
- added RGB6: LED_ABGR, marbastlib-various:MHT151RGBCT-RGB-Reverse-Mount-1206, B.Cu at (-292.1, -317.8)
- added RGB60: LED_ABGR, marbastlib-various:MHT151RGBCT-RGB-Reverse-Mount-1206, B.Cu at (-220.7, -255.9)
- added RGB61: LED_ABGR, marbastlib-various:MHT151RGBCT-RGB-Reverse-Mount-1206, B.Cu at (-201.6, -255.9)
- added RGB62: LED_ABGR, marbastlib-various:MHT151RGBCT-RGB-Reverse-Mount-1206, B.Cu at (-182.6, -255.9)
- added RGB63: LED_ABGR, marbastlib-various:MHT151RGBCT-RGB-Reverse-Mount-1206, B.Cu at (-163.5, -255.9)
- added RGB64: LED_ABGR, marbastlib-various:MHT151RGBCT-RGB-Reverse-Mount-1206, B.Cu at (-404.0, -236.9)
- added RGB65: LED_ABGR, marbastlib-various:MHT151RGBCT-RGB-Reverse-Mount-1206, B.Cu at (-382.6, -236.9)
- added RGB66: LED_ABGR, marbastlib-various:MHT151RGBCT-RGB-Reverse-Mount-1206, B.Cu at (-363.5, -236.9)
- added RGB67: LED_ABGR, marbastlib-various:MHT151RGBCT-RGB-Reverse-Mount-1206, B.Cu at (-344.5, -236.9)
- added RGB68: LED_ABGR, marbastlib-various:MHT151RGBCT-RGB-Reverse-Mount-1206, B.Cu at (-325.4, -236.9)
- added RGB69: LED_ABGR, marbastlib-various:MHT151RGBCT-RGB-Reverse-Mount-1206, B.Cu at (-306.4, -236.9)
- added RGB7: LED_ABGR, marbastlib-various:MHT151RGBCT-RGB-Reverse-Mount-1206, B.Cu at (-273.0, -317.8)
- added RGB70: LED_ABGR, marbastlib-various:MHT151RGBCT-RGB-Reverse-Mount-1206, B.Cu at (-287.3, -236.9)
- added RGB71: LED_ABGR, marbastlib-various:MHT151RGBCT-RGB-Reverse-Mount-1206, B.Cu at (-268.3, -236.9)
- added RGB72: LED_ABGR, marbastlib-various:MHT151RGBCT-RGB-Reverse-Mount-1206, B.Cu at (-249.2, -236.9)
- added RGB73: LED_ABGR, marbastlib-various:MHT151RGBCT-RGB-Reverse-Mount-1206, B.Cu at (-230.2, -236.9)
- added RGB74: LED_ABGR, marbastlib-various:MHT151RGBCT-RGB-Reverse-Mount-1206, B.Cu at (-211.1, -236.9)
- added RGB75: LED_ABGR, marbastlib-various:MHT151RGBCT-RGB-Reverse-Mount-1206, B.Cu at (-192.1, -236.9)
- added RGB76: LED_ABGR, marbastlib-various:MHT151RGBCT-RGB-Reverse-Mount-1206, B.Cu at (-156.4, -236.9)
- added RGB77: LED_ABGR, marbastlib-various:MHT151RGBCT-RGB-Reverse-Mount-1206, B.Cu at (-96.8, -236.9)
- added RGB78: LED_ABGR, marbastlib-various:MHT151RGBCT-RGB-Reverse-Mount-1206, B.Cu at (-401.6, -217.8)
- added RGB79: LED_ABGR, marbastlib-various:MHT151RGBCT-RGB-Reverse-Mount-1206, B.Cu at (-377.8, -217.8)
- added RGB8: LED_ABGR, marbastlib-various:MHT151RGBCT-RGB-Reverse-Mount-1206, B.Cu at (-244.5, -317.8)
- added RGB80: LED_ABGR, marbastlib-various:MHT151RGBCT-RGB-Reverse-Mount-1206, B.Cu at (-354.0, -217.8)
- added RGB82: LED_ABGR, marbastlib-various:MHT151RGBCT-RGB-Reverse-Mount-1206, B.Cu at (-211.1, -217.8)
- added RGB83: LED_ABGR, marbastlib-various:MHT151RGBCT-RGB-Reverse-Mount-1206, B.Cu at (-187.3, -217.8)
- added RGB84: LED_ABGR, marbastlib-various:MHT151RGBCT-RGB-Reverse-Mount-1206, B.Cu at (-168.3, -217.8)
- added RGB85: LED_ABGR, marbastlib-various:MHT151RGBCT-RGB-Reverse-Mount-1206, B.Cu at (-143.7, -217.8)
- added RGB86: LED_ABGR, marbastlib-various:MHT151RGBCT-RGB-Reverse-Mount-1206, B.Cu at (-115.9, -217.8)
- added RGB87: LED_ABGR, marbastlib-various:MHT151RGBCT-RGB-Reverse-Mount-1206, B.Cu at (-96.8, -217.8)
- added RGB88: LED_ABGR, marbastlib-various:MHT151RGBCT-RGB-Reverse-Mount-1206, B.Cu at (-77.8, -217.8)
- added RGB9: LED_ABGR, marbastlib-various:MHT151RGBCT-RGB-Reverse-Mount-1206, B.Cu at (-225.4, -317.8)
- added U3: IS313741A, marbastlib-various:QFN-60_EP_7x7_Pitch0.4mm, B.Cu at (-207.5, -184.7)
- C1, C2, C3: value 0.1uf -> 1uF
- C16, C17, C18, C19: value 0.1uf -> 100nF
- R8: value 100k -> 51k; footprint Capacitor_SMD:C_0402_1005Metric -> Resistor_SMD:R_0603_1608Metric
- btn1: renamed from btn2; moved to B.Cu
- moved J1 563.0 mm to (-231.8, -340.5), turned to 180 degrees
- moved R8 562.0 mm to (-212.3, -176.4)
- moved D33 535.3 mm to (-82.5, -280.5), turned to 0 degrees
- moved D32 523.0 mm to (-101.6, -280.5), turned to 0 degrees
- moved D30 512.6 mm to (-154.0, -280.5), turned to 0 degrees
- moved D8 510.2 mm to (-249.2, -304.3), turned to 0 degrees
- moved D10 506.5 mm to (-211.1, -304.3), turned to 0 degrees
- moved D48 505.6 mm to (-120.6, -261.5), turned to 0 degrees
- moved D29 505.5 mm to (-182.6, -280.5), turned to 0 degrees
- moved D50 504.4 mm to (-82.5, -261.5), turned to 0 degrees
- moved D47 498.8 mm to (-151.6, -258.3), turned to 0 degrees
- moved D6 495.9 mm to (-296.9, -304.3), turned to 0 degrees
- moved D77 491.3 mm to (-101.6, -223.4), turned to 0 degrees
- moved D7 490.5 mm to (-277.8, -304.3), turned to 0 degrees
- moved D2 489.7 mm to (-382.6, -304.3), turned to 0 degrees
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- renumbered C97 to C10, C98 to C11, C99 to C12, C100 to C13, C101 to C14, C102 to C15, C104 to C20, C105 to C21, C106 to C22, C107 to C23, C103 to C24, C91 to C4, C92 to C5, C93 to C6, C94 to C7, C95 to C8, C96 to C9, R4 to R12, R5 to R15, R2 to R4, R7 to R40, R6 to R41, R3 to R5, U3 to U4, U4 to U5, btn1 to btn2
Connections:
- C19 pad 1: +5V -> Net-(C19-Pad1)
- C19 pad 2: GND -> ~{SDB}
- R8 pad 1: +3V3 -> Net-(R8-Pad1)
- R8 pad 2: RGB -> CS3
- U2 pad 24: unconnected-(U2-Pad24) -> SWCLK
- U2 pad 25: unconnected-(U2-Pad25) -> SWDIO
- U2 pad 4: RGB -> unconnected-(U2-Pad4)
Other:
- board outline removed

Commit message: corrected top row layout
Parts:
- moved J1 25.3 mm to (-249.2, -322.3)
- moved D4 9.53 mm to (-335.0, -304.3)
- moved SW4 9.53 mm to (-330.2, -312.7)
- moved D2 9.52 mm to (-373.1, -304.3)
- moved D3 9.52 mm to (-354.0, -304.3)
- moved RGB2 9.52 mm to (-368.3, -317.8)
- moved RGB3 9.52 mm to (-349.2, -317.8)
- moved RGB4 9.52 mm to (-330.2, -317.8)
- moved SW2 9.52 mm to (-368.3, -312.7)
- moved SW3 9.52 mm to (-349.2, -312.7)
- moved D6 6.35 mm to (-290.5, -304.3)
- moved D7 6.35 mm to (-271.5, -304.3)
- moved RGB7 6.35 mm to (-266.7, -317.8)
- moved SW6 6.35 mm to (-285.8, -312.7)
- moved SW7 6.35 mm to (-266.7, -312.7)
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
Commit message: improved rgb schematic
Parts:
- removed RGB88: LED_ABGR, marbastlib-various:MHT151RGBCT-RGB-Reverse-Mount-1206
- added R42: 51k, Resistor_SMD:R_0603_1608Metric, B.Cu at (-173.8, -168.3)
- added R43: 20k, Resistor_SMD:R_0603_1608Metric, B.Cu at (-173.8, -170.8)
- added R44: 20k, Resistor_SMD:R_0603_1608Metric, B.Cu at (-177.8, -170.8)
- added R45: 51k, Resistor_SMD:R_0603_1608Metric, B.Cu at (-177.8, -168.3)
- added R46: 1k, Resistor_SMD:R_0402_1005Metric, B.Cu at (-181.3, -169.1)
- added R47: 1k, Resistor_SMD:R_0402_1005Metric, B.Cu at (-181.3, -171.0)
- added RGB81: LED_ABGR, marbastlib-various:MHT151RGBCT-RGB-Reverse-Mount-1206, B.Cu at (-211.1, -217.8)
- C10, C11, C12, C13, C14, C15, C4, C5, C9: value 100n -> 100nf
- C6, C8: value 1u -> 1uf
- J1: footprint Connector_USB:USB_C_Receptacle_HRO_TYPE-C-31-M-12 -> marbastlib-various:USB_C_Receptacle_HRO_TYPE-C-31-M-14
- R40, R41: value 1k -> 20k; footprint Resistor_SMD:R_0402_1005Metric -> Resistor_SMD:R_0603_1608Metric
- moved R15 167.6 mm to (-251.6, -318.1), turned to 0 degrees
- moved C20 165.2 mm to (-253.5, -310.4)
- moved R12 163.4 mm to (-247.3, -318.1), turned to 0 degrees
- moved U4 163.0 mm to (-254.0, -307.8), turned to 90 degrees
- moved C21 161.6 mm to (-254.5, -305.2)
- moved U1 160.8 mm to (-249.5, -315.0)
- moved C7 160.6 mm to (-254.5, -304.2), turned to 0 degrees
- moved F1 158.3 mm to (-254.0, -313.3), turned to -90 degrees
- moved btn1 111.1 mm to (-91.5, -254.9), turned to 90 degrees
- moved btn2 110.9 mm to (-91.4, -258.6), turned to 90 degrees
- moved U5 107.0 mm to (-108.9, -256.7)
- moved R41 92.4 mm to (-97.0, -258.6)
- moved R1 91.0 mm to (-97.0, -254.9), turned to 0 degrees
- moved J2 90.1 mm to (-121.8, -230.9)
- moved R5 88.6 mm to (-121.3, -253.5), turned to 90 degrees
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Connections:
- R40 pad 1: /XTAL_O -> Net-(R40-Pad1)
- R40 pad 2: XOUT -> CS31
- R41 pad 1: /~{USB_BOOT} -> Net-(R41-Pad1)
- R41 pad 2: SS -> CS32
- RGB10 pad 1: SW1 -> SW2
- RGB11 pad 1: SW2 -> SW3
- RGB12 pad 1: SW3 -> SW4
- RGB13 pad 1: SW4 -> SW5
- RGB14 pad 1: SW5 -> SW6
- RGB15 pad 1: SW6 -> SW7
- RGB16 pad 1: SW7 -> SW8
- RGB17 pad 1: SW8 -> SW1
- RGB17 pad 2: CS6 -> CS9
- RGB17 pad 3: CS5 -> CS8
- RGB17 pad 4: CS4 -> CS7
- RGB18 pad 1: SW9 -> SW2
- RGB18 pad 2: CS6 -> CS9
- RGB18 pad 3: CS5 -> CS8
- RGB18 pad 4: CS4 -> CS7
- RGB19 pad 1: SW1 -> SW3
- RGB20 pad 1: SW2 -> SW4
- RGB21 pad 1: SW3 -> SW5
- RGB22 pad 1: SW4 -> SW6
- RGB23 pad 1: SW5 -> SW7
- RGB24 pad 1: SW6 -> SW8
- RGB25 pad 1: SW7 -> SW9
- RGB26 pad 1: SW8 -> SW1
- RGB26 pad 2: CS9 -> CS12
- RGB26 pad 3: CS8 -> CS11
- RGB26 pad 4: CS7 -> CS10
- RGB27 pad 1: SW9 -> SW2
- RGB27 pad 2: CS9 -> CS12
- RGB27 pad 3: CS8 -> CS11
- RGB27 pad 4: CS7 -> CS10
- RGB28 pad 1: SW1 -> SW3
- RGB29 pad 1: SW2 -> SW4
- RGB30 pad 1: SW3 -> SW5
- RGB31 pad 1: SW4 -> SW6
- RGB32 pad 1: SW5 -> SW7
- RGB33 pad 1: SW6 -> SW8
- RGB34 pad 1: SW7 -> SW1
- RGB34 pad 2: CS12 -> CS15
- RGB34 pad 3: CS11 -> CS14
- RGB34 pad 4: CS10 -> CS13
- RGB35 pad 1: SW8 -> SW2
- RGB35 pad 2: CS12 -> CS15
- RGB35 pad 3: CS11 -> CS14
- RGB35 pad 4: CS10 -> CS13
- RGB36 pad 1: SW9 -> SW3
- RGB36 pad 2: CS12 -> CS15
- RGB36 pad 3: CS11 -> CS14
- RGB36 pad 4: CS10 -> CS13
- RGB37 pad 1: SW1 -> SW4
- RGB38 pad 1: SW2 -> SW5
- RGB39 pad 1: SW3 -> SW6
- RGB40 pad 1: SW4 -> SW7
- RGB41 pad 1: SW5 -> SW8
- RGB42 pad 1: SW6 -> SW9
- RGB43 pad 1: SW7 -> SW1
- RGB43 pad 2: CS15 -> CS18
- RGB43 pad 3: CS14 -> CS17
- RGB43 pad 4: CS13 -> CS16
- RGB44 pad 1: SW8 -> SW2
- RGB44 pad 2: CS15 -> CS18
- RGB44 pad 3: CS14 -> CS17
- RGB44 pad 4: CS13 -> CS16
- RGB45 pad 1: SW9 -> SW3
- RGB45 pad 2: CS15 -> CS18
- RGB45 pad 3: CS14 -> CS17
- RGB45 pad 4: CS13 -> CS16
- RGB46 pad 1: SW1 -> SW4
- RGB47 pad 1: SW2 -> SW5
- RGB48 pad 1: SW3 -> SW6
- RGB49 pad 1: SW4 -> SW7
- RGB50 pad 1: SW5 -> SW8
- RGB51 pad 1: SW6 -> SW1
- RGB51 pad 2: CS18 -> CS21
- RGB51 pad 3: CS17 -> CS20
- RGB51 pad 4: CS16 -> CS19
- RGB52 pad 1: SW7 -> SW2
- RGB52 pad 2: CS18 -> CS21
- RGB52 pad 3: CS17 -> CS20
- RGB52 pad 4: CS16 -> CS19
- RGB53 pad 1: SW8 -> SW3
- RGB53 pad 2: CS18 -> CS21
- RGB53 pad 3: CS17 -> CS20
- RGB53 pad 4: CS16 -> CS19
- RGB54 pad 1: SW9 -> SW4
- RGB54 pad 2: CS18 -> CS21
- RGB54 pad 3: CS17 -> CS20
- RGB54 pad 4: CS16 -> CS19
- RGB55 pad 1: SW1 -> SW5
- RGB56 pad 1: SW2 -> SW6
- RGB57 pad 1: SW3 -> SW7
- RGB58 pad 1: SW4 -> SW8
- RGB59 pad 1: SW5 -> SW9
- RGB60 pad 1: SW6 -> SW1
- RGB60 pad 2: CS21 -> CS24
- RGB60 pad 3: CS20 -> CS23
- RGB60 pad 4: CS19 -> CS22
- RGB61 pad 1: SW7 -> SW2
- RGB61 pad 2: CS21 -> CS24
- RGB61 pad 3: CS20 -> CS23
- RGB61 pad 4: CS19 -> CS22
- RGB62 pad 1: SW8 -> SW3
- RGB62 pad 2: CS21 -> CS24
- RGB62 pad 3: CS20 -> CS23
- RGB62 pad 4: CS19 -> CS22
- RGB63 pad 1: SW9 -> SW4
- RGB63 pad 2: CS21 -> CS24
- RGB63 pad 3: CS20 -> CS23
- RGB63 pad 4: CS19 -> CS22
- RGB64 pad 2: CS24 -> CS27
- RGB64 pad 3: CS23 -> CS26
- RGB64 pad 4: CS22 -> CS25
- RGB65 pad 2: CS24 -> CS27
- RGB65 pad 3: CS23 -> CS26
- RGB65 pad 4: CS22 -> CS25
- RGB66 pad 2: CS24 -> CS27
- RGB66 pad 3: CS23 -> CS26
- RGB66 pad 4: CS22 -> CS25
- RGB67 pad 2: CS24 -> CS27
- RGB67 pad 3: CS23 -> CS26
- RGB67 pad 4: CS22 -> CS25
- RGB68 pad 2: CS24 -> CS27
- RGB68 pad 3: CS23 -> CS26
- RGB68 pad 4: CS22 -> CS25
- RGB69 pad 2: CS24 -> CS27
- RGB69 pad 3: CS23 -> CS26
- RGB69 pad 4: CS22 -> CS25
- RGB70 pad 2: CS24 -> CS27
- RGB70 pad 3: CS23 -> CS26
- RGB70 pad 4: CS22 -> CS25
- RGB71 pad 2: CS24 -> CS27
- RGB71 pad 3: CS23 -> CS26
- RGB71 pad 4: CS22 -> CS25
- RGB72 pad 2: CS24 -> CS27
- RGB72 pad 3: CS23 -> CS26
- RGB72 pad 4: CS22 -> CS25
- RGB73 pad 2: CS27 -> CS30
- RGB73 pad 3: CS26 -> CS29
- RGB73 pad 4: CS25 -> CS28
- RGB74 pad 2: CS27 -> CS30
- RGB74 pad 3: CS26 -> CS29
- RGB74 pad 4: CS25 -> CS28
- RGB75 pad 2: CS27 -> CS30
- RGB75 pad 3: CS26 -> CS29
- RGB75 pad 4: CS25 -> CS28
- RGB76 pad 2: CS27 -> CS30
- RGB76 pad 3: CS26 -> CS29
- RGB76 pad 4: CS25 -> CS28
- RGB77 pad 1: SW5 -> SW7
- RGB77 pad 2: CS27 -> CS30
- RGB77 pad 3: CS26 -> CS29
- RGB77 pad 4: CS25 -> CS28
- RGB78 pad 1: SW6 -> SW1
- RGB78 pad 2: CS27 -> CS33
- RGB78 pad 3: CS26 -> CS32
- RGB78 pad 4: CS25 -> CS31
- RGB79 pad 1: SW7 -> SW2
- RGB79 pad 2: CS27 -> CS33
- RGB79 pad 3: CS26 -> CS32
- RGB79 pad 4: CS25 -> CS31
- RGB80 pad 1: SW8 -> SW3
- RGB80 pad 2: CS27 -> CS33
- RGB80 pad 3: CS26 -> CS32
- RGB80 pad 4: CS25 -> CS31
- RGB82 pad 1: SW9 -> SW2
- RGB82 pad 2: CS27 -> CS36
- RGB82 pad 3: CS26 -> CS35
- RGB82 pad 4: CS25 -> CS34
- RGB83 pad 1: SW1 -> SW3
- RGB83 pad 2: CS30 -> CS36
- RGB83 pad 3: CS29 -> CS35
- RGB83 pad 4: CS28 -> CS34
- RGB84 pad 1: SW2 -> SW4
- RGB84 pad 2: CS30 -> CS36
- RGB84 pad 3: CS29 -> CS35
- RGB84 pad 4: CS28 -> CS34
- RGB85 pad 1: SW3 -> SW5
- RGB85 pad 2: CS30 -> CS36
- RGB85 pad 3: CS29 -> CS35
- RGB85 pad 4: CS28 -> CS34
- RGB86 pad 1: SW4 -> SW7
- RGB86 pad 2: CS30 -> CS36
- RGB86 pad 3: CS29 -> CS35
- RGB86 pad 4: CS28 -> CS34
- RGB87 pad 1: SW5 -> SW8
- RGB87 pad 2: CS30 -> CS36
- RGB87 pad 3: CS29 -> CS35
- RGB87 pad 4: CS28 -> CS34
- U1 pad 3: DN -> DP
- U1 pad 4: DP -> DN
- U3 pad 1: unconnected-(U3-Pad1) -> Net-(R43-Pad1)
- U3 pad 2: unconnected-(U3-Pad2) -> Net-(R44-Pad1)
- U3 pad 3: unconnected-(U3-Pad3) -> Net-(R45-Pad1)
- U3 pad 58: unconnected-(U3-Pad58) -> Net-(R40-Pad1)
- U3 pad 59: unconnected-(U3-Pad59) -> Net-(R41-Pad1)
- U3 pad 60: unconnected-(U3-Pad60) -> Net-(R42-Pad1)
Routing:
- net +3V3: track 0.00 -> 242.1 mm, vias 0 -> 3
- net CS2: track 0.00 -> 198.2 mm
- net CS3: track 0.00 -> 196.7 mm, vias 0 -> 16
- net CS1: track 0.00 -> 194.4 mm
- net DN: track 0.00 -> 192.8 mm, vias 0 -> 1
- net DP: track 0.00 -> 191.9 mm, vias 0 -> 1
- net ROW0: track 0.00 -> 191.8 mm, vias 0 -> 4
- net CS12: track 0.00 -> 168.9 mm, vias 0 -> 14
- net CS11: track 0.00 -> 167.5 mm, vias 0 -> 2
- net CS9: track 0.00 -> 165.6 mm, vias 0 -> 16
- net CS8: track 0.00 -> 164.6 mm
- net CS10: track 0.00 -> 163.5 mm, vias 0 -> 2
- net CS7: track 0.00 -> 162.3 mm
- net CS5: track 0.00 -> 135.2 mm
- net CS6: track 0.00 -> 134.9 mm, vias 0 -> 12
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- added copper zone on B.Cu, net +3V3
Other:
- board outline added: 347.7 x 125.4 mm

Commit message: small fixes
Parts:
- moved R41 130.7 mm to (-200.1, -178.2)
- moved R47 121.5 mm to (-97.1, -258.6)
- moved R40 106.6 mm to (-208.1, -184.0), turned to 0 degrees
- moved R46 95.8 mm to (-117.9, -240.9), turned to 45 degrees
Connections:
- RGB2 pad 1: SW2 -> SW3
- RGB3 pad 1: SW3 -> SW4
- RGB4 pad 1: SW4 -> SW5
- RGB5 pad 1: SW5 -> SW6
- RGB6 pad 1: SW6 -> SW7
- RGB7 pad 1: SW7 -> SW8
- RGB8 pad 1: SW8 -> SW9
- RGB9 pad 1: SW9 -> SW1
- RGB9 pad 2: CS3 -> CS6
- RGB9 pad 3: CS2 -> CS5
- RGB9 pad 4: CS1 -> CS4
Routing:
- net CS21: track 0.00 -> 173.4 mm, vias 0 -> 16
- net CS20: track 0.00 -> 171.5 mm
- net CS15: track 0.00 -> 171.5 mm, vias 0 -> 16
- net CS14: track 0.00 -> 169.8 mm
- net CS27: track 0.00 -> 169.3 mm, vias 0 -> 16
- net CS26: track 0.00 -> 167.4 mm
- net CS19: track 0.00 -> 167.3 mm
- net CS18: track 0.00 -> 167.3 mm, vias 0 -> 14
- net CS17: track 0.00 -> 164.9 mm, vias 0 -> 2
- net CS25: track 0.00 -> 162.9 mm
- net CS16: track 0.00 -> 161.5 mm, vias 0 -> 2
- net CS36: track 0.00 -> 144.3 mm, vias 0 -> 12
- net CS35: track 0.00 -> 142.6 mm
- net CS30: track 0.00 -> 141.4 mm, vias 0 -> 8
- net CS29: track 0.00 -> 140.1 mm
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
Commit message: wiring components
Connections:
- U2 pad 13: ROW3 -> COL12
- U2 pad 15: ROW1 -> COL16
- U2 pad 16: ROW0 -> COL15
- U2 pad 17: ROW5 -> ROW4
- U2 pad 18: ROW4 -> ROW5
- U2 pad 2: COL16 -> ROW0
- U2 pad 27: COL12 -> COL10
- U2 pad 29: COL10 -> ROW3
- U2 pad 3: COL15 -> ROW1
Routing:
- net SW7: track 0.00 -> 430.8 mm, vias 0 -> 14
- net SW8: track 0.00 -> 420.1 mm, vias 0 -> 12
- net SW6: track 0.00 -> 370.5 mm, vias 0 -> 10
- net ROW5: track 0.00 -> 369.6 mm, vias 0 -> 2
- net ROW4: track 0.00 -> 337.2 mm, vias 0 -> 2
- net ROW1: track 0.00 -> 331.1 mm, vias 0 -> 2
- net ROW2: track 0.00 -> 329.5 mm, vias 0 -> 2
- net SW3: track 135.7 -> 462.5 mm, vias 6 -> 14
- net SW2: track 107.5 -> 433.1 mm, vias 5 -> 13
- net SW1: track 135.8 -> 450.0 mm, vias 6 -> 14
- net SW5: track 117.3 -> 427.9 mm, vias 5 -> 11
- net SW4: track 111.4 -> 421.8 mm, vias 5 -> 13
- net ROW3: track 0.00 -> 304.6 mm
- net COL11: track 0.00 -> 152.7 mm, vias 0 -> 10
- net ROW0: track 191.8 -> 335.8 mm
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
Commit message: more routing done
Parts:
- moved C10 1.32 mm to (-122.2, -240.1)
- moved C4 1.32 mm to (-122.2, -241.2)
- moved C22 1.13 mm to (-116.5, -237.4)
- moved R46 1.13 mm to (-119.0, -241.4)
- moved C23 1.13 mm to (-119.9, -237.1)
- moved Y1 1.13 mm to (-118.1, -239.0)
- moved C11 0.17 mm to (-125.1, -251.0)
- moved C14 0.17 mm to (-125.1, -250.0)
Connections:
- U2 pad 12: COL14 -> unconnected-(U2-Pad12)
- U2 pad 14: ROW2 -> COL14
- U2 pad 31: COL8 -> COL7
- U2 pad 32: COL7 -> COL8
- U2 pad 34: COL6 -> COL13
- U2 pad 35: COL5 -> COL6
- U2 pad 36: COL4 -> COL5
- U2 pad 37: COL3 -> COL4
- U2 pad 38: COL2 -> COL3
- U2 pad 39: COL13 -> COL2
- U2 pad 5: unconnected-(U2-Pad5) -> ROW2
Routing:
- net COL1: track 100.3 -> 466.3 mm, vias 8 -> 10
- net COL0: track 125.8 -> 491.4 mm, vias 10 -> 11
- net COL2: track 131.8 -> 465.4 mm, vias 10 -> 11
- net COL3: track 108.3 -> 426.2 mm, vias 8 -> 9
- net COL4: track 107.9 -> 402.8 mm, vias 8 -> 9
- net COL5: track 120.1 -> 399.1 mm, vias 8 -> 9
- net COL6: track 119.2 -> 378.2 mm, vias 8 -> 9
- net ROW0: track 335.8 -> 440.1 mm
- net COL16: track 100.0 -> 147.6 mm
- net ROW1: track 331.1 -> 372.2 mm, vias 2 -> 4
- net ROW2: track 329.5 -> 355.5 mm, vias 2 -> 4
- net COL15: track 125.0 -> 148.9 mm, vias 8 -> 9
- net COL13: track 134.8 -> 152.3 mm
- net GND: track 42.8 -> 52.7 mm
- net COL14: track 109.4 -> 116.1 mm, vias 6 -> 7
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