File: rp2040-ISO-keyboard-pcb.kicad_pcb (KiCad board)
At the start: 2 copper layers, 347.7 x 125.4 mm, 349 parts, among them J1 USB_C_Receptacle_USB2.0, J2 Conn_01x04, SW1 SW_HS, SW10 SW_HS, SW11 SW_HS, SW12 SW_HS, SW13 SW_HS, SW14 SW_HS, SW15 SW_HS, SW16 SW_HS, SW17 SW_HS, SW18 SW_HS, SW19 SW_HS, SW2 SW_HS, SW20 SW_HS, SW21 SW_HS, SW22 SW_HS, SW23 SW_HS, SW24 SW_HS, SW25 SW_HS, SW26 SW_HS, SW27 SW_HS, SW28 SW_HS, SW29 SW_HS, SW3 SW_HS, SW30 SW_HS, SW31 SW_HS, SW32 SW_HS, SW33 SW_HS, SW34 SW_HS, SW35 SW_HS, SW36 SW_HS, SW37 SW_HS, SW38 SW_HS, SW39 SW_HS, SW4 SW_HS, SW40 SW_HS, SW41 SW_HS, SW42 SW_HS, SW43 SW_HS, SW44 SW_HS, SW45 SW_HS, SW46 SW_HS, SW47 SW_HS, SW48 SW_HS, SW49 SW_HS, SW5 SW_HS, SW50 SW_HS, SW51 SW_HS, SW52 SW_HS, SW53 SW_HS, SW54 SW_HS, SW55 SW_HS, SW56 SW_HS, SW57 SW_HS, SW58 SW_HS, SW59 SW_HS, SW6 SW_HS, SW60 SW_HS, SW61 SW_HS, SW62 SW_HS, SW63 SW_HS, SW64 SW_HS, SW65 SW_HS, SW66 SW_HS, SW67 SW_HS, SW68 SW_HS, SW69 SW_HS, SW7 SW_HS, SW70 SW_HS, SW71 SW_HS, SW72 SW_HS, SW73 SW_HS, SW74 SW_HS, SW75 SW_HS, SW76 SW_HS, SW77 SW_HS, SW78 SW_HS, SW79 SW_HS, SW8 SW_HS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

Commit message: sw pins done
Parts:
- moved R42 102.9 mm to (-269.6, -206.1)
- moved R9 73.6 mm to (-273.0, -199.5)
- moved R41 68.5 mm to (-262.6, -206.2), turned to 0 degrees
- moved R40 62.5 mm to (-266.5, -206.1)
- moved R8 61.7 mm to (-269.4, -199.7)
- moved R6 56.6 mm to (-261.1, -199.9), turned to 0 degrees
- moved R7 47.9 mm to (-264.9, -199.5)
- moved C18 18.7 mm to (-261.6, -208.5), turned to -90 degrees
- moved R3 17.2 mm to (-253.0, -214.8), turned to 0 degrees
- moved R2 16.6 mm to (-253.0, -216.3), turned to 0 degrees
- moved R18 14.4 mm to (-243.8, -199.4)
- moved C19 13.8 mm to (-253.5, -213.5)
- moved C17 12.1 mm to (-254.1, -208.9), turned to -90 degrees
- moved C16 11.9 mm to (-255.2, -208.9), turned to -90 degrees
- moved C3 11.9 mm to (-260.6, -208.5), turned to -90 degrees
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Connections:
- R40 pad 1: Net-(R40-Pad1) -> Net-(U3-Pad27)
- R41 pad 1: Net-(R41-Pad1) -> Net-(U3-Pad26)
- R42 pad 1: Net-(R42-Pad1) -> Net-(U3-Pad28)
- U2 pad 27: COL10 -> unconnected-(U2-Pad27)
- U2 pad 28: COL11 -> ROW3
- U2 pad 29: ROW3 -> COL11
- U2 pad 30: COL9 -> COL10
- U2 pad 31: COL7 -> COL9
- U2 pad 34: COL13 -> COL7
- U2 pad 4: unconnected-(U2-Pad4) -> ROW2
- U2 pad 5: ROW2 -> COL13
- U3 pad 16: SW1 -> SW9
- U3 pad 17: SW2 -> SW6
- U3 pad 18: SW3 -> SW7
- U3 pad 19: SW4 -> SW8
- U3 pad 20: SW5 -> SW1
- U3 pad 21: SW6 -> SW2
- U3 pad 22: SW7 -> SW3
- U3 pad 23: SW8 -> SW4
- U3 pad 24: SW9 -> SW5
- U3 pad 26: Net-(R6-Pad1) -> Net-(U3-Pad26)
- U3 pad 27: Net-(R7-Pad1) -> Net-(U3-Pad27)
- U3 pad 28: Net-(R8-Pad1) -> Net-(U3-Pad28)
- U3 pad 58: Net-(R40-Pad1) -> Net-(R6-Pad1)
- U3 pad 59: Net-(R41-Pad1) -> Net-(R7-Pad1)
- U3 pad 60: Net-(R42-Pad1) -> Net-(R8-Pad1)
Routing:
- net SW8: track 420.1 -> 618.2 mm, vias 12 -> 13
- net SW7: track 430.8 -> 617.7 mm, vias 14 -> 15
- net SW1: track 450.0 -> 604.0 mm, vias 14 -> 15
- net COL7: track 118.7 -> 259.4 mm, vias 8 -> 9
- net COL12: track 140.5 -> 280.3 mm, vias 10 -> 12
- net SW2: track 433.1 -> 565.8 mm, vias 13 -> 14
- net COL8: track 117.4 -> 242.0 mm, vias 8 -> 9
- net CS31: track 49.9 -> 168.8 mm, vias 0 -> 2
- net SW3: track 462.5 -> 568.7 mm, vias 14 -> 16
- net COL9: track 120.0 -> 225.8 mm, vias 8 -> 9
- net SW4: track 421.8 -> 526.0 mm, vias 13 -> 14
- net CS32: track 50.3 -> 153.9 mm, vias 0 -> 2
- net SW5: track 429.2 -> 518.8 mm, vias 11 -> 12
- net CS33: track 51.2 -> 138.9 mm
- net COL10: track 140.9 -> 228.2 mm, vias 10 -> 11
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
Commit message: some more CS pins done
Parts:
- moved R34 77.4 mm to (-267.8, -211.3)
- moved R35 71.8 mm to (-266.8, -212.9)
- moved R30 64.8 mm to (-270.9, -211.3)
- moved R22 61.4 mm to (-275.6, -207.2), turned to -90 degrees
- moved R24 60.9 mm to (-271.8, -207.2), turned to -90 degrees
- moved R29 57.1 mm to (-268.2, -209.7)
- moved R23 56.2 mm to (-274.1, -207.2), turned to -90 degrees
- moved R36 54.0 mm to (-269.9, -213.5)
- moved R28 52.3 mm to (-271.2, -209.7)
- moved R16 17.9 mm to (-236.1, -194.4)
- moved R19 17.9 mm to (-238.9, -191.9)
- moved R27 17.9 mm to (-230.2, -185.1)
- moved R33 17.9 mm to (-218.2, -182.1)
- moved R44 17.9 mm to (-191.8, -182.1)
- moved R11 17.9 mm to (-218.2, -187.1)
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Connections:
- R16 pad 1: Net-(R16-Pad1) -> Net-(U3-Pad45)
- R17 pad 1: Net-(R17-Pad1) -> Net-(U3-Pad46)
- R18 pad 1: Net-(R18-Pad1) -> Net-(U3-Pad47)
- R28 pad 1: Net-(R28-Pad1) -> Net-(U3-Pad32)
- R29 pad 1: Net-(R29-Pad1) -> Net-(U3-Pad33)
- R30 pad 1: Net-(R30-Pad1) -> Net-(U3-Pad34)
- R9 pad 1: Net-(R9-Pad1) -> Net-(U3-Pad51)
- U3 pad 29: Net-(R9-Pad1) -> Net-(R22-Pad1)
- U3 pad 30: Net-(R11-Pad1) -> Net-(R24-Pad1)
- U3 pad 31: Net-(R14-Pad1) -> Net-(R23-Pad1)
- U3 pad 32: Net-(R16-Pad1) -> Net-(U3-Pad32)
- U3 pad 33: Net-(R17-Pad1) -> Net-(U3-Pad33)
- U3 pad 34: Net-(R18-Pad1) -> Net-(U3-Pad34)
- U3 pad 35: Net-(R19-Pad1) -> Net-(R34-Pad1)
- U3 pad 37: Net-(R20-Pad1) -> Net-(R35-Pad1)
- U3 pad 38: Net-(R21-Pad1) -> Net-(R36-Pad1)
- U3 pad 39: Net-(R22-Pad1) -> Net-(R19-Pad1)
- U3 pad 40: Net-(R23-Pad1) -> Net-(R20-Pad1)
- U3 pad 41: Net-(R24-Pad1) -> Net-(R21-Pad1)
- U3 pad 45: Net-(R28-Pad1) -> Net-(U3-Pad45)
- U3 pad 46: Net-(R29-Pad1) -> Net-(U3-Pad46)
- U3 pad 47: Net-(R30-Pad1) -> Net-(U3-Pad47)
- U3 pad 51: Net-(R34-Pad1) -> Net-(U3-Pad51)
- U3 pad 52: Net-(R35-Pad1) -> Net-(R11-Pad1)
- U3 pad 53: Net-(R36-Pad1) -> Net-(R14-Pad1)
Routing:
- net CS15: track 171.5 -> 394.5 mm, vias 16 -> 20
- net CS14: track 169.8 -> 383.8 mm
- net CS13: track 164.5 -> 377.6 mm
- net CS20: track 171.5 -> 375.2 mm
- net CS21: track 173.4 -> 374.9 mm, vias 16 -> 18
- net CS19: track 167.3 -> 365.9 mm, vias 0 -> 2
- net CS26: track 167.4 -> 344.7 mm
- net CS25: track 162.9 -> 340.0 mm
- net CS27: track 169.3 -> 343.8 mm, vias 16 -> 18
- net CS31: track 168.8 -> 151.0 mm
- net Net-(R22-Pad1): track 0.00 -> 16.9 mm
- net Net-(R23-Pad1): track 0.00 -> 14.5 mm
- net Net-(R24-Pad1): track 0.00 -> 11.7 mm
- net Net-(U3-Pad32): track 0.00 -> 10.00 mm
- net Net-(U3-Pad34): track 0.00 -> 9.48 mm
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
Commit message: more routing
Parts:
- moved R17 59.6 mm to (-273.7, -215.1), turned to -90 degrees
- moved R16 41.6 mm to (-272.2, -215.1), turned to -90 degrees
- moved R18 30.0 mm to (-269.0, -215.7)
- moved R6 22.3 mm to (-273.6, -218.4), turned to -90 degrees
- moved R8 21.8 mm to (-277.4, -220.0)
- moved R7 21.5 mm to (-275.1, -218.4), turned to -90 degrees
- moved D42 5.13 mm to (-248.4, -261.7), turned to 180 degrees
- moved D25 4.81 mm to (-258.3, -280.7), turned to 180 degrees
- moved C19 0.20 mm to (-253.3, -213.5)
Connections:
- R16 pad 1: Net-(U3-Pad45) -> Net-(U3-Pad40)
- R17 pad 1: Net-(U3-Pad46) -> Net-(U3-Pad39)
- R18 pad 1: Net-(U3-Pad47) -> Net-(U3-Pad41)
- U3 pad 39: Net-(R19-Pad1) -> Net-(U3-Pad39)
- U3 pad 40: Net-(R20-Pad1) -> Net-(U3-Pad40)
- U3 pad 41: Net-(R21-Pad1) -> Net-(U3-Pad41)
- U3 pad 42: Net-(R25-Pad1) -> Net-(R7-Pad1)
- U3 pad 43: Net-(R26-Pad1) -> Net-(R6-Pad1)
- U3 pad 44: Net-(R27-Pad1) -> Net-(R8-Pad1)
- U3 pad 45: Net-(U3-Pad45) -> Net-(R19-Pad1)
- U3 pad 46: Net-(U3-Pad46) -> Net-(R20-Pad1)
- U3 pad 47: Net-(U3-Pad47) -> Net-(R21-Pad1)
- U3 pad 58: Net-(R6-Pad1) -> Net-(R25-Pad1)
- U3 pad 59: Net-(R7-Pad1) -> Net-(R26-Pad1)
- U3 pad 60: Net-(R8-Pad1) -> Net-(R27-Pad1)
Routing:
- net CS1: track 174.4 -> 345.4 mm, vias 0 -> 2
- net CS7: track 162.3 -> 328.0 mm, vias 0 -> 4
- net CS2: track 177.6 -> 341.3 mm, vias 0 -> 2
- net CS9: track 165.6 -> 328.6 mm, vias 16 -> 18
- net CS3: track 182.5 -> 345.0 mm, vias 14 -> 15
- net CS8: track 164.6 -> 325.6 mm, vias 0 -> 4
- net +5V: track 32.1 -> 102.8 mm
- net +3V3: track 240.4 -> 305.4 mm
- net Net-(R8-Pad1): track 0.00 -> 15.2 mm
- net Net-(R7-Pad1): track 0.00 -> 13.2 mm
- net Net-(U3-Pad39): track 0.00 -> 11.8 mm
- net Net-(R6-Pad1): track 0.00 -> 11.7 mm
- net Net-(U3-Pad40): track 0.00 -> 10.1 mm
- net COL7: track 259.4 -> 266.7 mm, vias 9 -> 10
- net GND: track 52.7 -> 59.4 mm, vias 23 -> 27
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
Commit message: added more routing
Parts:
- moved R11 66.1 mm to (-273.8, -222.8)
- moved R14 59.7 mm to (-273.8, -221.2)
- moved R26 58.7 mm to (-261.8, -221.4)
- moved R31 56.2 mm to (-254.6, -221.1), turned to 0 degrees
- moved R33 50.5 mm to (-253.8, -217.9), turned to 0 degrees
- moved R20 47.0 mm to (-269.5, -221.6), turned to 90 degrees
- moved R21 46.7 mm to (-267.9, -221.2), turned to 90 degrees
- moved R25 45.8 mm to (-265.6, -220.6)
- moved R27 45.6 mm to (-258.8, -220.6), turned to 0 degrees
- moved R32 45.2 mm to (-253.2, -219.5), turned to 0 degrees
- moved R19 44.2 mm to (-271.1, -222.0), turned to 90 degrees
- moved R9 22.5 mm to (-277.4, -221.6)
- moved D72 4.15 mm to (-254.2, -223.6), turned to 180 degrees
- moved D59 4.11 mm to (-244.8, -242.6), turned to 180 degrees
Connections:
- U3 pad 45: Net-(R19-Pad1) -> Net-(R9-Pad1)
- U3 pad 46: Net-(R20-Pad1) -> Net-(R14-Pad1)
- U3 pad 47: Net-(R21-Pad1) -> Net-(R11-Pad1)
- U3 pad 48: Net-(R31-Pad1) -> Net-(R19-Pad1)
- U3 pad 49: Net-(R32-Pad1) -> Net-(R20-Pad1)
- U3 pad 50: Net-(R33-Pad1) -> Net-(R21-Pad1)
- U3 pad 51: Net-(R9-Pad1) -> Net-(R25-Pad1)
- U3 pad 52: Net-(R11-Pad1) -> Net-(R26-Pad1)
- U3 pad 53: Net-(R14-Pad1) -> Net-(R27-Pad1)
- U3 pad 58: Net-(R25-Pad1) -> Net-(R31-Pad1)
- U3 pad 59: Net-(R26-Pad1) -> Net-(R32-Pad1)
- U3 pad 60: Net-(R27-Pad1) -> Net-(R33-Pad1)
Routing:
- net CS4: track 152.2 -> 306.4 mm, vias 0 -> 2
- net CS6: track 158.9 -> 312.1 mm, vias 14 -> 16
- net CS5: track 155.0 -> 303.7 mm, vias 0 -> 2
- net CS12: track 168.9 -> 285.7 mm, vias 14 -> 16
- net CS10: track 164.1 -> 280.5 mm, vias 2 -> 4
- net CS11: track 167.5 -> 282.4 mm, vias 2 -> 4
- net CS16: track 161.5 -> 252.9 mm, vias 2 -> 4
- net CS17: track 164.6 -> 254.1 mm, vias 2 -> 4
- net CS18: track 168.1 -> 252.8 mm, vias 14 -> 16
- net CS22: track 60.2 -> 125.9 mm, vias 0 -> 2
- net CS24: track 62.8 -> 127.4 mm, vias 6 -> 8
- net CS23: track 61.4 -> 122.4 mm, vias 0 -> 2
- net +5V: track 102.8 -> 153.2 mm, vias 2 -> 3
- net +3V3: track 305.4 -> 346.8 mm
- net Net-(R9-Pad1): track 0.00 -> 16.0 mm
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
Commit message: routing finished
Parts:
- added C0: 22uf/10v, Capacitor_Tantalum_SMD:CP_EIA-3216-18_Kemet-A, B.Cu at (-254.8, -206.9)
- moved R43 57.0 mm to (-233.9, -215.5), turned to 90 degrees
- moved R45 52.7 mm to (-230.2, -215.5), turned to 90 degrees
- moved R44 52.4 mm to (-232.1, -215.5), turned to 90 degrees
- moved R37 36.4 mm to (-233.9, -220.7), turned to 90 degrees
- moved R38 31.4 mm to (-232.1, -220.7), turned to 90 degrees
- moved R39 21.4 mm to (-230.2, -220.7), turned to 90 degrees
- moved R33 4.63 mm to (-249.8, -220.2), turned to -90 degrees
- moved R2 4.32 mm to (-249.5, -213.8), turned to 90 degrees
- moved C16 3.03 mm to (-252.3, -208.2)
- moved C1 3.03 mm to (-253.2, -208.2)
- moved C17 3.03 mm to (-251.1, -208.3)
- moved C2 3.03 mm to (-250.1, -208.3)
- moved R3 2.21 mm to (-251.0, -213.8), turned to 90 degrees
- moved R13 1.00 mm to (-252.2, -210.1)
- moved R31 0.99 mm to (-255.6, -221.3)
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Connections:
- U3 pad 1: Net-(R43-Pad1) -> Net-(R37-Pad1)
- U3 pad 2: Net-(R44-Pad1) -> Net-(R38-Pad1)
- U3 pad 3: Net-(R45-Pad1) -> Net-(R39-Pad1)
- U3 pad 4: unconnected-(U3-Pad4) -> Net-(R43-Pad1)
- U3 pad 5: unconnected-(U3-Pad5) -> Net-(R44-Pad1)
- U3 pad 54: Net-(R37-Pad1) -> unconnected-(U3-Pad54)
- U3 pad 56: Net-(R38-Pad1) -> unconnected-(U3-Pad56)
- U3 pad 57: Net-(R39-Pad1) -> unconnected-(U3-Pad57)
- U3 pad 6: unconnected-(U3-Pad6) -> Net-(R45-Pad1)
Routing:
- net Net-(R45-Pad1): track 0.00 -> 29.5 mm, vias 0 -> 2
- net Net-(R39-Pad1): track 0.00 -> 28.8 mm, vias 0 -> 2
- net Net-(R44-Pad1): track 0.00 -> 27.6 mm, vias 0 -> 2
- net Net-(R38-Pad1): track 0.00 -> 26.8 mm, vias 0 -> 2
- net Net-(R37-Pad1): track 0.00 -> 25.3 mm, vias 0 -> 2
- net Net-(R43-Pad1): track 0.00 -> 25.1 mm, vias 0 -> 2
- net SWDIO: track 0.00 -> 24.8 mm, vias 0 -> 2
- net CS36: track 144.3 -> 166.7 mm
- net CS34: track 138.2 -> 160.2 mm
- net SWCLK: track 0.00 -> 21.5 mm, vias 0 -> 2
- net CS35: track 142.6 -> 162.8 mm, vias 0 -> 2
- net CS28: track 139.3 -> 159.0 mm
- net +3V3: track 346.8 -> 366.4 mm, vias 2 -> 3
- net CS29: track 140.1 -> 157.8 mm, vias 0 -> 2
- net CS30: track 141.4 -> 157.5 mm
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